File: ATSAMx21.kicad_pcb (KiCad board)
At the start: 2 copper layers, 50 x 55 mm, 0 parts

Commit message: Updated Schematic and Created Laytout
Parts:
- added C1: 22pF, Capacitors_SMD:C_1206_HandSoldering, B.Cu at (119.4, 78.7)
- added C10: 100nF, Capacitors_SMD:C_1206_HandSoldering, B.Cu at (132.1, 99.1)
- added C11: 100nF-Close, Capacitors_SMD:C_1206_HandSoldering, B.Cu at (128.3, 88.9)
- added C12: 10uF, Capacitors_SMD:C_1206_HandSoldering, B.Cu at (116.8, 64.8)
- added C13: 100nF, Capacitors_SMD:C_1206_HandSoldering, B.Cu at (125.7, 71.1)
- added C14: 10uF, Capacitors_SMD:C_1206_HandSoldering, B.Cu at (125.7, 73.7)
- added C15: 10uF, Capacitors_SMD:C_1206_HandSoldering, B.Cu at (127.0, 64.8)
- added C16: 100nF, Capacitors_SMD:C_1206_HandSoldering, B.Cu at (127.0, 62.2)
- added C2: 22pF, Capacitors_SMD:C_1206_HandSoldering, B.Cu at (118.1, 85.1)
- added C3: 22pF, Capacitors_SMD:C_1206_HandSoldering, B.Cu at (138.4, 104.1)
- added C4: 22pF, Capacitors_SMD:C_1206_HandSoldering, B.Cu at (147.3, 104.1)
- added C5: 1uF, Capacitors_SMD:C_1206_HandSoldering, B.Cu at (135.9, 76.2)
- added C6: 1uFC, Capacitors_SMD:C_1206_HandSoldering, B.Cu at (139.7, 82.5)
- added C7: 100nF-Close, Capacitors_SMD:C_1206_HandSoldering, B.Cu at (132.1, 82.5)
- added C8: 10uF, Capacitors_SMD:C_1206_HandSoldering, F.Cu at (134.6, 82.5)
- added C9: 100nF, Capacitors_SMD:C_1206_HandSoldering, B.Cu at (144.8, 85.1)
- added D1: 1N4001, Diodes_SMD:D_SMB_Handsoldering, F.Cu at (116.8, 71.1)
- added J1: PORTA_1, Pin_Headers:Pin_Header_Straight_1x08_Pitch2.54mm, F.Cu at (113.0, 78.7)
- added J2: PORTA_2, Pin_Headers:Pin_Header_Straight_1x08_Pitch2.54mm, F.Cu at (125.7, 111.8)
- added J3: PORTA_4, Pin_Headers:Pin_Header_Straight_1x06_Pitch2.54mm, F.Cu at (148.8, 75.5)
- added J4: PORTA_3, Pin_Headers:Pin_Header_Straight_1x08_Pitch2.54mm, F.Cu at (157.5, 111.8)
- added J5: PORTB, Pin_Headers:Pin_Header_Straight_1x08_Pitch2.54mm, F.Cu at (157.4, 69.3)
- added J6: PWR, Pin_Headers:Pin_Header_Straight_1x02_Pitch2.54mm, F.Cu at (113.0, 66.0)
- added J7: JTAG, Pin_Headers:Pin_Header_Straight_1x05_Pitch2.54mm, F.Cu at (132.1, 63.5)
- added R1: 10k, Resistors_SMD:R_1206_HandSoldering, B.Cu at (135.9, 80.0)
- added R2: 1k, Resistors_SMD:R_1206_HandSoldering, B.Cu at (134.6, 66.0)
- added U1: ATSAMx21G, ATSAMD21G18A-AU:QFP50P900X900X120-48N, F.Cu at (135.0, 90.0)
- added U2: AP111733, TO_SOT_Packages_SMD:SOT-223, F.Cu at (123.2, 64.8)
- added Y1: XOSC32K, Crystals:Crystal_HC49-4H_Vertical, F.Cu at (121.9, 81.3)
- added Y2: XOSC, Crystals:Crystal_HC49-4H_Vertical, F.Cu at (139.7, 100.3)
Routing:
- net GND: track 0.00 -> 172.0 mm, vias 0 -> 2
- net VDD: track 0.00 -> 95.6 mm, vias 0 -> 3
- net SWDIO: track 0.00 -> 48.9 mm, vias 0 -> 2
- net SWDCLK: track 0.00 -> 45.2 mm
- net Net-(J5-Pad1): track 0.00 -> 40.0 mm, vias 0 -> 1
- net Net-(J5-Pad2): track 0.00 -> 39.3 mm, vias 0 -> 1
- net Net-(J5-Pad6): track 0.00 -> 38.1 mm, vias 0 -> 1
- net Net-(J5-Pad4): track 0.00 -> 38.1 mm, vias 0 -> 1
- net Net-(J5-Pad5): track 0.00 -> 37.8 mm, vias 0 -> 1
- net Net-(J5-Pad3): track 0.00 -> 36.7 mm, vias 0 -> 1
- net /MCU/PA25: track 0.00 -> 31.6 mm, vias 0 -> 2
- net /MCU/PA0: track 0.00 -> 29.2 mm
- net /MCU/PA1: track 0.00 -> 29.1 mm
- net /MCU/PA28: track 0.00 -> 28.6 mm
- net /MCU/PA16: track 0.00 -> 28.3 mm
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- added copper zone on B.Cu, net GND
- added copper zone on F.Cu, net GND

Commit message: Added Gerbers
Parts:
- added REF**: 1pin, Connectors:1pin, F.Cu at (156.0, 64.0)
- added REF**: 1pin, Connectors:1pin, F.Cu at (114.0, 111.0)
- added REF**: 1pin, Connectors:1pin, F.Cu at (150.0, 111.0)
- added REF**: 1pin, Connectors:1pin, F.Cu at (120.0, 75.0)
Other:
- net class Default: clearance 0.2 -> 0.01524; trace_width 0.25 -> 0.01524; via_dia 0.6 -> 0.01524; via_drill 0.4 -> 0.01016
- rule trace_clearance: 0.2 -> 0.01524
- rule trace_min: 0.2 -> 0.01524
- rule via_min_drill: 0.3 -> 0.01016
- rule via_min_size: 0.4 -> 0.01524
- board text added: "+"
- board text added: "-"
- board text added: "0"
- board text added: "1"
- board text added: "10"
- board text added: "11"
- board text added: "12"
- board text added: "13"
- board text added: "14"
- board text added: "15"
- board text added: "16"
- board text added: "17"
- board text added: "18"
- board text added: "19"
- board text added: "2"
- board text added: "20"
- board text added: "2018-02 Ver. A.0"
- board text added: "21"
- board text added: "22"
- board text added: "23"
- board text added: "24"
- board text added: "25"
- board text added: "27"
- board text added: "28"
- board text added: "3"
- board text added: "30"
- board text added: "31"
- board text added: "4"
- board text added: "5"
- board text added: "6"
- board text added: "7"
- board text added: "8"
- board text added: "9"
- board text added: "SAMx21Gxx Demo Board"
- board text added: "SWD"

Commit message: Generated gerbers
Parts:
- renumbered REF** to ?
Changed lines of the file:
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@@
     (links 92)
     (no_connects 2)
-    (area 109.239524 59.0711 161.270477 115.565)
+    (area 109.824284 59.65586 160.685717 115.075001)
     (thickness 1.6)
     (drawings 52)
@@
     (visible_elements 7FFFFFFF)
     (pcbplotparams
-      (layerselection 0x00030_80000001)
-      (usegerberextensions false)
+      (layerselection 0x010f0_80000001)
+      (usegerberextensions true)
       (excludeedgelayer true)
       (linewidth 0.100000)
@@
       (psa4output false)
       (plotreference true)
-      (plotvalue true)
+      (plotvalue false)
       (plotinvisibletext false)
       (padsonsilk false)
@@
       (outputformat 1)
       (mirror false)
-      (drillshape 1)
+      (drillshape 0)
       (scaleselection 1)
       (outputdirectory ""))
@@
     (descr "module 1 pin (ou trou mecanique de percage)")
     (tags DEV)
-    (fp_text reference REF** (at 0 -3.048) (layer F.SilkS)
+    (fp_text reference "" (at 0 -3.048) (layer F.SilkS)
       (effects (font (size 1 1) (thickness 0.15)))
     )
@@
     (descr "module 1 pin (ou trou mecanique de percage)")
     (tags DEV)
-    (fp_text reference REF** (at 0 -3.048) (layer F.SilkS)
+    (fp_text reference "" (at 0 -3.048) (layer F.SilkS)
       (effects (font (size 1 1) (thickness 0.15)))
     )
@@
     (descr "module 1 pin (ou trou mecanique de percage)")
     (tags DEV)
-    (fp_text reference REF** (at 0 -3.048) (layer F.SilkS)
+    (fp_text reference "" (at 0 -3.048) (layer F.SilkS)
       (effects (font (size 1 1) (thickness 0.15)))
     )
@@
   (gr_line (start 116.3574 71.86168) (end 117.06606 71.15302) (angle 90) (layer F.SilkS) (width 0.2))
   (gr_line (start 116.3574 70.39864) (end 116.3574 71.86168) (angle 90) (layer F.SilkS) (width 0.2))
-  (gr_text "2018-02\nVer. A.0" (at 117.475 107.95) (layer F.SilkS)
+  (gr_text "2018-02\nVer. A.0" (at 120.8532 105.8672) (layer F.SilkS)
     (effects (font (size 1.5 1.5) (thickness 0.3)))
   )
@@
     (effects (font (size 1.5 1.5) (thickness 0.3)))
   )
-  (gr_text "SAMx21Gxx\nDemo Board" (at 118.11 102.87) (layer F.SilkS)
+  (gr_text "SAMx21Gxx\nDemo Board" (at 121.8692 100.584) (layer F.SilkS)
     (effects (font (size 1.5 1.5) (thickness 0.3)))
   )
